File: jianjia.kicad_pcb (KiCad board)
At the start: 2 copper layers, 90 x 55 mm, 62 parts, among them J1 PROG, J2 USB, Q1 BSS138, Q2 SI2301CDS, Q3 SI2301CDS, SW1 RESET, SW2 BOOT/CONFIG, U1 ESP32-S3-WROOM-2, U2 AC073TC1_FH34SRJ-50S-0.5SH, U3 CN3130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

Commit message: rev1: tune PCB
Parts:
- D6: moved to F.Cu
- moved C28 29.5 mm to (132.8, 66.2), turned to 180 degrees
- moved R10 28.5 mm to (129.3, 69.2), turned to 90 degrees
- moved R11 27.6 mm to (135.9, 69.1)
- moved U3 27.3 mm to (132.7, 69.0)
- moved D6 19.9 mm to (139.0, 69.0), turned to 0 degrees
- moved D5 18.8 mm to (135.3, 64.0)
- moved R12 17.5 mm to (139.7, 66.7)
- moved R9 17.0 mm to (133.0, 61.3)
- moved Q3 16.3 mm to (136.8, 59.9)
- moved C27 13.7 mm to (139.7, 64.8), turned to 0 degrees
- moved SW2 1.72 mm to (132.1, 53.7)
Routing:
- net GND: track 124.6 -> 155.9 mm, vias 14 -> 82
- net +BATT: track 128.5 -> 144.4 mm, vias 8 -> 9
- net +5V: track 27.3 -> 19.4 mm
- net CHG_VIN: track 10.9 -> 16.8 mm, vias 0 -> 2
- net Net-(D6-K): track 3.55 -> 6.35 mm, vias 1 -> 0
- net USB_DP: track 33.2 -> 35.9 mm
- net USB_DM: track 35.6 -> 38.4 mm
- net DISP_SCLK: track 44.6 -> 43.9 mm
- net Net-(D6-A): track 3.19 -> 2.61 mm, vias 1 -> 0
- net Net-(U3-ISET): track 2.53 -> 2.02 mm
- net BOOT: track 29.3 -> 29.5 mm, vias 0 -> 2
